Commit message: Gets Velocity Controller Working

File: ros2_ws/src/rover_control/urdf/driverover.urdf.xacro (robot description, xacro)
@@ -77,19 +77,71 @@
     </joint>
   </xacro:macro>
-<xacro:wheel name="wheel1" x_wheel="0.205359" y_wheel="0.2" tilt_sign="1"/>
+  <xacro:wheel name="front_left_wheel" x_wheel="-0.7" y_wheel="0.5" tilt_sign="-1"/>
+  <xacro:wheel name="front_right_wheel" x_wheel="0.7" y_wheel="0.5" tilt_sign="1"/>
+  <xacro:wheel name="middle_left_wheel" x_wheel="-0.7" y_wheel="0" tilt_sign="-1"/>
+  <xacro:wheel name="middle_right_wheel" x_wheel="0.7" y_wheel="0" tilt_sign="1"/>
+  <xacro:wheel name="rear_left_wheel" x_wheel="-0.7" y_wheel="-0.5" tilt_sign="-1"/>
+  <xacro:wheel name="rear_right_wheel" x_wheel="0.7" y_wheel="-0.5" tilt_sign="1"/>
   <joint name="chasis_base_joint" type="fixed">
     <parent link="base_link"/>
     <child link="chasis_link"/>
-    <origin xyz="-0.1 0 0"/>
+    <origin xyz="0 0 0"/>
   </joint>
-  <joint name="chasis_to_wheel1" type="continuous">
-    <parent link="chasis_link"/>
-    <child link="wheel1"/>
-    <origin xyz="0.205359 0.2 0.125" rpy="0 0 0"/>
-    <axis xyz="0 0 1"/>
-  </joint>
+  <ros2_control name="GazeboSystem" type="system">
+    <hardware>
+      <plugin>gazebo_ros2_control/GazeboSystem</plugin>
+    </hardware>
+    <joint name="front_left_wheel_joint">
+      <command_interface name="velocity">
+        <param name="min">-10</param>
+        <param name="max">10</param>
+      </command_interface>
+      <state_interface name="position" />
+      <state_interface name="velocity" />
+    </joint>
+    <joint name="front_right_wheel_joint">
+      <command_interface name="velocity">
+        <param name="min">-10</param>
+        <param name="max">10</param>
+      </command_interface>
+      <state_interface name="velocity" />
+      <state_interface name="position" />
+    </joint>
+    <joint name="middle_left_wheel_joint">
+      <command_interface name="velocity">
+        <param name="min">-10</param>
+        <param name="max">10</param>
+      </command_interface>
+      <state_interface name="position" />
+      <state_interface name="velocity" />
+    </joint>
+    <joint name="middle_right_wheel_joint">
+      <command_interface name="velocity">
+        <param name="min">-10</param>
+        <param name="max">10</param>
+      </command_interface>
+      <state_interface name="velocity" />
+      <state_interface name="position" />
+    </joint>
+    <joint name="rear_left_wheel_joint">
+      <command_interface name="velocity">
+        <param name="min">-10</param>
+        <param name="max">10</param>
+      </command_interface>
+      <state_interface name="velocity" />
+      <state_interface name="position" />
+    </joint>
+    <joint name="rear_right_wheel_joint">
+      <command_interface name="velocity">
+        <param name="min">-10</param>
+        <param name="max">10</param>
+      </command_interface>
+      <state_interface name="velocity" />
+      <state_interface name="position" />
+    </joint>
+  </ros2_control>
   <gazebo>
     <plugin filename="libgazebo_ros2_control.so" name="gazebo_ros2_control">
-      <parameters>$(find rover_control)/config/my_controller.yaml</parameters>
+      <parameters>$(find rover_control)/config/rover_control.yaml</parameters>
     </plugin>
   </gazebo>

Commit message: Adds effort controller

File: ros2_ws/src/rover_control/urdf/driverover.urdf.xacro (robot description, xacro)
@@ -70,4 +70,14 @@
       </inertial>
     </link>
+    <!-- <transmission name="transmission_name">
+      <type>transmission_interface/SimpleTransmission</type>
+      <joint name="joint_name">
+        <hardwareInterface>hardware_interface/PositionJointInterface</hardwareInterface>
+      </joint>
+      <actuator name="actuator_name">
+        <mechanicalReduction>1.0</mechanicalReduction>
+        <hardwareInterface>hardware_interface/PositionJointInterface</hardwareInterface>
+      </actuator>
+    </transmission> -->
     <joint name="${name}_joint" type="continuous">
       <parent link="base_link" />
@@ -88,9 +98,10 @@
     <origin xyz="0 0 0"/>
   </joint>
-  <ros2_control name="GazeboSystem" type="system">
-    <hardware>
-      <plugin>gazebo_ros2_control/GazeboSystem</plugin>
-    </hardware>
-    <joint name="front_left_wheel_joint">
+  <xacro:macro name="wheel_joint" params="name">
+    <joint name="${name}">
+      <command_interface name="effort">
+        <param name="min">-10</param>
+        <param name="max">10</param>
+      </command_interface>
       <command_interface name="velocity">
         <param name="min">-10</param>
@@ -100,44 +111,15 @@
       <state_interface name="velocity" />
     </joint>
-    <joint name="front_right_wheel_joint">
-      <command_interface name="velocity">
-        <param name="min">-10</param>
-        <param name="max">10</param>
-      </command_interface>
-      <state_interface name="velocity" />
-      <state_interface name="position" />
-    </joint>
-    <joint name="middle_left_wheel_joint">
-      <command_interface name="velocity">
-        <param name="min">-10</param>
-        <param name="max">10</param>
-      </command_interface>
-      <state_interface name="position" />
-      <state_interface name="velocity" />
-    </joint>
-    <joint name="middle_right_wheel_joint">
-      <command_interface name="velocity">
-        <param name="min">-10</param>
-        <param name="max">10</param>
-      </command_interface>
-      <state_interface name="velocity" />
-      <state_interface name="position" />
-    </joint>
-    <joint name="rear_left_wheel_joint">
-      <command_interface name="velocity">
-        <param name="min">-10</param>
-        <param name="max">10</param>
-      </command_interface>
-      <state_interface name="velocity" />
-      <state_interface name="position" />
-    </joint>
-    <joint name="rear_right_wheel_joint">
-      <command_interface name="velocity">
-        <param name="min">-10</param>
-        <param name="max">10</param>
-      </command_interface>
-      <state_interface name="velocity" />
-      <state_interface name="position" />
-    </joint>
+  </xacro:macro>
+  <ros2_control name="GazeboSystem" type="system">
+    <hardware>
+      <plugin>gazebo_ros2_control/GazeboSystem</plugin>
+    </hardware>
+    <xacro:wheel_joint name="front_left_wheel_joint"/>
+    <xacro:wheel_joint name="front_right_wheel_joint"/>
+    <xacro:wheel_joint name="middle_left_wheel_joint"/>
+    <xacro:wheel_joint name="middle_right_wheel_joint"/>
+    <xacro:wheel_joint name="rear_left_wheel_joint"/>
+    <xacro:wheel_joint name="rear_right_wheel_joint"/>
   </ros2_control>
   <gazebo>
